Commit message: gazebo

File: training_ws1/src/test_robot_description/urdf/test_robot.urdf (robot description, URDF)
Before this commit: robot test_robot, 4 links, 3 joints
Links:
- added link lwheel_link, mass 0.1; collision cylinder length=0.01 radius=0.5; visual cylinder length=0.01 radius=0.05
Joints:
- added joint lwheel_j: type continuous, parent body_link, child lwheel_link, origin xyz=0.1 0.12 0 rpy=0 0 0, axis 0 1 0
- joint rwheel_j: origin xyz=0.1 0.12 0 rpy=0 0 0 -> xyz=0.1 -0.12 0 rpy=0 0 0

File: training_ws2/src/test_robot_description/urdf/test_robot.urdf.xacro (robot description, xacro)
@@ -39,5 +39,5 @@
             <cylinder length="${wheel_width}" radius="${wheel_radius}"/>
         </geometry>
-        <origin rpy="${pi} 0 0" xyz="0 0 0"/>
+        <origin rpy="${pi/2} 0 0" xyz="0 0 0"/>
         <material name="black">
             <color rgba="0 0 0 1"/>
@@ -48,5 +48,5 @@
             <cylinder length="${wheel_width}" radius="${wheel_radius}"/>
         </geometry>
-        <origin rpy="${pi} 0 0" xyz="0 0 0"/>
+        <origin rpy="${pi/2} 0 0" xyz="0 0 0"/>
         </collision>
         <inertial>
